Commit message: added scene factory, car modeling correct, and single stage okay

File: artifacts/student_vehicle_assets/import_smoke/student_fwd_vehicle.urdf (robot description, URDF)
Before this commit: robot student_fwd_vehicle, 11 links, 10 joints
Links:
- link base_link: mass 520 -> 1800; geometry collision box size=4 2 1; visual box size=4 2 1
- link front_left_steer_link: geometry visual sphere radius=0.045
- link front_left_suspension_link: geometry visual box size=0.08 0.05 0.175
- link front_left_wheel_link: mass 18 -> 20; geometry collision cylinder length=0.15 radius=0.35; visual cylinder length=0.15 radius=0.35
- link front_right_steer_link: geometry visual sphere radius=0.045
- link front_right_suspension_link: geometry visual box size=0.08 0.05 0.175
- link front_right_wheel_link: mass 18 -> 20; geometry collision cylinder length=0.15 radius=0.35; visual cylinder length=0.15 radius=0.35
- link rear_left_suspension_link: geometry visual box size=0.08 0.05 0.175
- link rear_left_wheel_link: mass 18 -> 20; geometry collision cylinder length=0.15 radius=0.35; visual cylinder length=0.15 radius=0.35
- link rear_right_suspension_link: geometry visual box size=0.08 0.05 0.175
- link rear_right_wheel_link: mass 18 -> 20; geometry collision cylinder length=0.15 radius=0.35; visual cylinder length=0.15 radius=0.35
Joints:
- joint front_left_steer_joint: limit lower=-0.523598776 upper=0.523598776 effort=1200 velocity=4 -> lower=-0.558505361 upper=0.558505361 effort=1200 velocity=4; origin xyz=0 0 -0.04 rpy=0 0 0 -> xyz=0 0 -0.0875 rpy=0 0 0
- joint front_left_suspension_joint: limit lower=-0.08 upper=0.08 effort=15000 velocity=3 -> lower=-0.175 upper=0.175 effort=15000 velocity=3; origin xyz=0.64 0.46 0.03 rpy=0 0 0 -> xyz=1.3 1 -0.325 rpy=0 0 0
- joint front_left_wheel_joint: origin xyz=0 0 -0.02 rpy=0 0 0 -> xyz=0 0 -0.0875 rpy=0 0 0
- joint front_right_steer_joint: limit lower=-0.523598776 upper=0.523598776 effort=1200 velocity=4 -> lower=-0.558505361 upper=0.558505361 effort=1200 velocity=4; origin xyz=0 0 -0.04 rpy=0 0 0 -> xyz=0 0 -0.0875 rpy=0 0 0
- joint front_right_suspension_joint: limit lower=-0.08 upper=0.08 effort=15000 velocity=3 -> lower=-0.175 upper=0.175 effort=15000 velocity=3; origin xyz=0.64 -0.46 0.03 rpy=0 0 0 -> xyz=1.3 -1 -0.325 rpy=0 0 0
- joint front_right_wheel_joint: origin xyz=0 0 -0.02 rpy=0 0 0 -> xyz=0 0 -0.0875 rpy=0 0 0
- joint rear_left_suspension_joint: limit lower=-0.08 upper=0.08 effort=15000 velocity=3 -> lower=-0.175 upper=0.175 effort=15000 velocity=3; origin xyz=-0.64 0.46 0.03 rpy=0 0 0 -> xyz=-1.3 1 -0.325 rpy=0 0 0
- joint rear_left_wheel_joint: origin xyz=0 0 -0.02 rpy=0 0 0 -> xyz=0 0 -0.0875 rpy=0 0 0
- joint rear_right_suspension_joint: limit lower=-0.08 upper=0.08 effort=15000 velocity=3 -> lower=-0.175 upper=0.175 effort=15000 velocity=3; origin xyz=-0.64 -0.46 0.03 rpy=0 0 0 -> xyz=-1.3 -1 -0.325 rpy=0 0 0
- joint rear_right_wheel_joint: origin xyz=0 0 -0.02 rpy=0 0 0 -> xyz=0 0 -0.0875 rpy=0 0 0
